File: Arduino Header Wing/Arduino Header Wing.kicad_pcb (KiCad board)
At the start: 2 copper layers, 87 x 64.8 mm, 24 parts, among them U1 TXB0104, U2 TXB0104, U3 TXB0104, U4 TXB0104, U5 TXB0104

Commit message: Quetzalcoatl V1.0
Digital Snake Wing
Parts:
- moved U5 43.8 mm to (248.4, 77.2), turned to 270 degrees
- moved C11 30.6 mm to (285.0, 69.6)
- moved U3 28.7 mm to (248.4, 67.1), turned to 270 degrees
- moved U4 28.2 mm to (258.1, 89.9), turned to 270 degrees
- moved ADC1 27.7 mm to (247.4, 89.4), turned to 90 degrees
- moved C1 20.2 mm to (263.1, 70.1)
- moved U1 14.5 mm to (248.4, 56.9), turned to 270 degrees
- moved U2 10.2 mm to (258.1, 79.8), turned to 270 degrees
Connections:
- PAP1 pad 1: N-000006 -> (no net)
- PAP1 pad 10: N-0000055 -> N-000009
- PAP1 pad 11: N-0000052 -> N-000005
- PAP1 pad 12: N-0000056 -> N-000008
- PAP1 pad 13: (no net) -> N-000007
- PAP1 pad 14: (no net) -> N-000006
- PAP1 pad 15: (no net) -> N-0000012
- PAP1 pad 16: (no net) -> N-0000011
- PAP1 pad 2: N-0000015 (its old number) -> (no net)
- PAP1 pad 22: (no net) -> +3.3V
- PAP1 pad 23: +3.3V -> (no net)
- PAP1 pad 3: N-0000059 -> (no net)
- PAP1 pad 4: N-0000060 (its old number) -> (no net)
- PAP1 pad 5: N-0000058 -> N-0000062
- PAP1 pad 6: N-0000062 -> N-0000064
- PAP1 pad 8: N-0000053 -> N-0000023
- PAP1 pad 9: N-0000054 -> N-0000010
- U1 pad 2: N-0000060 (its old number) -> N-000007
- U1 pad 3: N-0000059 -> N-000006
- U1 pad 4: N-0000015 (its old number) -> N-0000012
- U1 pad 5: N-000006 -> N-0000011
- U3 pad 2: N-0000053 -> N-0000010
- U3 pad 3: N-0000063 -> N-000009
- U3 pad 4: N-0000062 -> N-000005
- U3 pad 5: N-0000058 -> N-000008
- U5 pad 2: N-0000056 -> N-0000062
- U5 pad 3: N-0000052 -> N-0000064
- U5 pad 4: N-0000055 -> N-0000063
- U5 pad 5: N-0000054 -> N-0000023
Routing:
- net N-00000106: track 6.69 -> 33.5 mm
- net N-0000099: track 7.21 -> 30.4 mm
- net N-00000100: track 7.74 -> 27.4 mm
- net N-000004: track 7.34 -> 20.7 mm
- net N-000003: track 6.81 -> 17.6 mm
- net N-0000091: track 8.53 -> 0.00 mm
- net N-0000090: track 8.00 -> 0.00 mm
- net N-000002: track 6.92 -> 14.5 mm
- net N-0000089: track 7.48 -> 0.00 mm
- net N-0000093: track 6.95 -> 0.00 mm
- net N-0000092: track 6.79 -> 0.00 mm
- net N-000001: track 7.45 -> 11.5 mm
