File: Arduino Header Wing/Arduino Header Wing.sch (KiCad schematic (older format))
At the start: 24 parts, among them U1 TXB0104, U2 TXB0104, U3 TXB0104, U4 TXB0104, U5 TXB0104

Commit message: Quetzalcoatl V1.0
Digital Snake Wing
Connections:
- net +3.3V: now also PAP1.22 (3V3); no longer PAP1.23 (2V5)
- net at PAP1.1 (0): no longer U1.5 (A4)
- net at PAP1.10 (9): now also U3.3 (A2); no longer U5.4 (A3)
- net at PAP1.11 (10): now also U3.4 (A3); no longer U5.3 (A2)
- net at PAP1.12 (11): now also U3.5 (A4); no longer U5.2 (A1)
- net at PAP1.13 (12): now also U1.2 (A1)
- net at PAP1.14 (13): now also U1.3 (A2)
- net at PAP1.15 (14): now also U1.4 (A3)
- net at PAP1.16 (15): now also U1.5 (A4)
- net at PAP1.2 (1): no longer U1.4 (A3)
- net at PAP1.3 (2): no longer U1.3 (A2)
- net at PAP1.4 (3): no longer U1.2 (A1)
- net at PAP1.5 (4): now also U5.2 (A1); no longer U3.5 (A4)
- net at PAP1.6 (5): now also U5.3 (A2); no longer U3.4 (A3)
- net at PAP1.7 (6): now also U5.4 (A3); no longer U3.3 (A2)
- net at PAP1.8 (7): now also U5.5 (A4); no longer U3.2 (A1)
- net at PAP1.9 (8): now also U3.2 (A1); no longer U5.5 (A4)
- no-connect marks 15 -> 11
Changed lines of the file:
@@
-$EndComp
-$Comp
-L PAPILIO_WINGS PAP1
-U 1 1 53E3DC81
-P 9950 2800
-F 0 "PAP1" H 9900 3550 60  0000 C CNN
-F 1 "PAPILIO_WINGS" H 9950 3650 60  0000 C CNN
-F 2 "~" H 9600 3650 60  0000 C CNN
-F 3 "~" H 9600 3650 60  0000 C CNN
-	1    9950 2800
-	1    0    0    -1
 $EndComp
 $Comp
@@
 $EndComp
 $Comp
-L GND #PWR24
+L GND #PWR01
 U 1 1 53E3EBF8
 P 1950 6200
-F 0 "#PWR24" H 1950 6200 30  0001 C CNN
+F 0 "#PWR01" H 1950 6200 30  0001 C CNN
 F 1 "GND" H 1950 6130 30  0001 C CNN
 F 2 "~" H 1950 6200 60  0000 C CNN
@@
 $EndComp
 $Comp
-L +5V #PWR3
+L +5V #PWR02
 U 1 1 53E3EEF2
 P 4950 2300
-F 0 "#PWR3" H 4950 2390 20  0001 C CNN
+F 0 "#PWR02" H 4950 2390 20  0001 C CNN
 F 1 "+5V" H 4950 2390 30  0000 C CNN
 F 2 "~" H 4950 2300 60  0000 C CNN
@@
 $EndComp
 $Comp
-L +3.3V #PWR4
+L +3.3V #PWR03
 U 1 1 53E3EF6A
 P 5050 2300
-F 0 "#PWR4" H 5050 2260 30  0001 C CNN
+F 0 "#PWR03" H 5050 2260 30  0001 C CNN
 F 1 "+3.3V" H 5100 2400 30  0000 C CNN
 F 2 "~" H 5050 2300 60  0000 C CNN
@@
 $EndComp
 $Comp
-L GND #PWR20
+L GND #PWR04
 U 1 1 53E3F587
 P 3350 4450
-F 0 "#PWR20" H 3350 4450 30  0001 C CNN
+F 0 "#PWR04" H 3350 4450 30  0001 C CNN
 F 1 "GND" H 3350 4380 30  0001 C CNN
 F 2 "~" H 3350 4450 60  0000 C CNN
@@
 $EndComp
 $Comp
-L GND #PWR12
+L GND #PWR05
 U 1 1 53E3F61B
 P 3300 3400
-F 0 "#PWR12" H 3300 3400 30  0001 C CNN
+F 0 "#PWR05" H 3300 3400 30  0001 C CNN
 F 1 "GND" H 3300 3330 30  0001 C CNN
 F 2 "~" H 3300 3400 60  0000 C CNN
@@
 $EndComp
 $Comp
-L +3.3V #PWR5
+L +3.3V #PWR06
 U 1 1 53E3F6B0
 P 3350 2450
-F 0 "#PWR5" H 3350 2410 30  0001 C CNN
+F 0 "#PWR06" H 3350 2410 30  0001 C CNN
 F 1 "+3.3V" H 3350 2560 30  0000 C CNN
 F 2 "~" H 3350 2450 60  0000 C CNN
@@
 $EndComp
 $Comp
-L +3.3V #PWR14
+L +3.3V #PWR07
 U 1 1 53E3F748
 P 3300 3650
-F 0 "#PWR14" H 3300 3610 30  0001 C CNN
+F 0 "#PWR07" H 3300 3610 30  0001 C CNN
 F 1 "+3.3V" H 3300 3760 30  0000 C CNN
 F 2 "~" H 3300 3650 60  0000 C CNN
@@
 NoConn ~ 3400 4250
 $Comp
-L +5V #PWR15
+L +5V #PWR08
 U 1 1 53E3F7E1
 P 4400 3650
-F 0 "#PWR15" H 4400 3740 20  0001 C CNN
+F 0 "#PWR08" H 4400 3740 20  0001 C CNN
 F 1 "+5V" H 4400 3740 30  0000 C CNN
 F 2 "~" H 4400 3650 60  0000 C CNN
@@
 NoConn ~ 7150 2300
 $Comp
-L +5V #PWR9
+L +5V #PWR09
 U 1 1 53E3F9A6
 P 7200 2950
-F 0 "#PWR9" H 7200 3040 20  0001 C CNN
+F 0 "#PWR09" H 7200 3040 20  0001 C CNN
 F 1 "+5V" H 7200 3040 30  0000 C CNN
 F 2 "~" H 7200 2950 60  0000 C CNN
@@
 NoConn ~ 7150 3300
 $Comp
-L GND #PWR11
+L GND #PWR010
 U 1 1 53E3FAE4
 P 8250 3250
-F 0 "#PWR11" H 8250 3250 30  0001 C CNN
+F 0 "#PWR010" H 8250 3250 30  0001 C CNN
 F 1 "GND" H 8250 3180 30  0001 C CNN
 F 2 "~" H 8250 3250 60  0000 C CNN
@@
 $EndComp
 $Comp
-L +3.3V #PWR10
+L +3.3V #PWR011
 U 1 1 53E3FB89
 P 8050 2950
-F 0 "#PWR10" H 8050 2910 30  0001 C CNN
+F 0 "#PWR011" H 8050 2910 30  0001 C CNN
 F 1 "+3.3V" H 8050 3060 30  0000 C CNN
 F 2 "~" H 8050 2950 60  0000 C CNN
@@
 $EndComp
 $Comp
-L +5V #PWR16
+L +5V #PWR012
 U 1 1 53E400AB
 P 7200 4050
-F 0 "#PWR16" H 7200 4140 20  0001 C CNN
+F 0 "#PWR012" H 7200 4140 20  0001 C CNN
 F 1 "+5V" H 7200 4140 30  0000 C CNN
 F 2 "~" H 7200 4050 60  0000 C CNN
@@
 $EndComp
 $Comp
-L +3.3V #PWR17
+L +3.3V #PWR013
 U 1 1 53E400B1
 P 8050 4050
-F 0 "#PWR17" H 8050 4010 30  0001 C CNN
+F 0 "#PWR013" H 8050 4010 30  0001 C CNN
 F 1 "+3.3V" H 8050 4160 30  0000 C CNN
 F 2 "~" H 8050 4050 60  0000 C CNN
@@
 $EndComp
 $Comp
-L GND #PWR19
+L GND #PWR014
 U 1 1 53E402A1
 P 8250 4200
-F 0 "#PWR19" H 8250 4200 30  0001 C CNN
+F 0 "#PWR014" H 8250 4200 30  0001 C CNN
 F 1 "GND" H 8250 4130 30  0001 C CNN
 F 2 "~" H 8250 4200 60  0000 C CNN
@@
 $EndComp
 $Comp
-L +3.3V #PWR22
+L +3.3V #PWR015
 U 1 1 53E402B0
 P 8050 5000
-F 0 "#PWR22" H 8050 4960 30  0001 C CNN
+F 0 "#PWR015" H 8050 4960 30  0001 C CNN
 F 1 "+3.3V" H 8050 5110 30  0000 C CNN
 F 2 "~" H 8050 5000 60  0000 C CNN
@@
 $EndComp
 $Comp
-L +5V #PWR21
+L +5V #PWR016
 U 1 1 53E402BF
 P 7200 5000
-F 0 "#PWR21" H 7200 5090 20  0001 C CNN
+F 0 "#PWR016" H 7200 5090 20  0001 C CNN
 F 1 "+5V" H 7200 5090 30  0000 C CNN
 F 2 "~" H 7200 5000 60  0000 C CNN
@@
 $EndComp
 $Comp
-L +5V #PWR6
+L +5V #PWR017
 U 1 1 53E404CE
 P 4450 2600
-F 0 "#PWR6" H 4450 2690 20  0001 C CNN
+F 0 "#PWR017" H 4450 2690 20  0001 C CNN
 F 1 "+5V" H 4450 2690 30  0000 C CNN
 F 2 "~" H 4450 2600 60  0000 C CNN
@@
 $EndComp
 $Comp
-L GND #PWR18
+L GND #PWR018
 U 1 1 53E4091B
 P 700 4200
-F 0 "#PWR18" H 700 4200 30  0001 C CNN
+F 0 "#PWR018" H 700 4200 30  0001 C CNN
 F 1 "GND" H 700 4130 30  0001 C CNN
 F 2 "~" H 700 4200 60  0000 C CNN
@@
 $EndComp
 $Comp
-L +3.3V #PWR8
+L +3.3V #PWR019
 U 1 1 53E40934
 P 850 2850
-F 0 "#PWR8" H 850 2810 30  0001 C CNN
+F 0 "#PWR019" H 850 2810 30  0001 C CNN
 F 1 "+3.3V" H 850 2960 30  0000 C CNN
 F 2 "~" H 850 2850 60  0000 C CNN
@@
 $EndComp
 $Comp
-L +5V #PWR7
+L +5V #PWR020
 U 1 1 53E409FD
 P 750 2850
-F 0 "#PWR7" H 750 2940 20  0001 C CNN
+F 0 "#PWR020" H 750 2940 20  0001 C CNN
 F 1 "+5V" H 750 2940 30  0000 C CNN
 F 2 "~" H 750 2850 60  0000 C CNN
@@
 Connection ~ 6050 5550
 $Comp
-L +5V #PWR23
+L +5V #PWR021
 U 1 1 53E42A26
 P 6050 5500
-F 0 "#PWR23" H 6050 5590 20  0001 C CNN
+F 0 "#PWR021" H 6050 5590 20  0001 C CNN
 F 1 "+5V" H 6050 5590 30  0000 C CNN
 F 2 "~" H 6050 5500 60  0000 C CNN
@@
 Connection ~ 6200 6350
 $Comp
-L +3.3V #PWR25
+L +3.3V #PWR022
 U 1 1 53E42B55
 P 6200 6300
-F 0 "#PWR25" H 6200 6260 30  0001 C CNN
+F 0 "#PWR022" H 6200 6260 30  0001 C CNN
 F 1 "+3.3V" H 6200 6410 30  0000 C CNN
 F 2 "~" H 6200 6300 60  0000 C CNN
@@
 Connection ~ 5050 6850
 $Comp
-L GND #PWR26
+L GND #PWR023
 U 1 1 53E42D89
 P 5050 6900
-F 0 "#PWR26" H 5050 6900 30  0001 C CNN
+F 0 "#PWR023" H 5050 6900 30  0001 C CNN
 F 1 "GND" H 5050 6830 30  0001 C CNN
 F 2 "~" H 5050 6900 60  0000 C CNN
@@
 $EndComp
 Wire Wire Line
-	10550 2200 10600 2200
-Wire Wire Line
-	10600 2200 10600 3400
-Wire Wire Line
-	10600 3000 10550 3000
-Wire Wire Line
-	10650 3200 10550 3200
-Wire Wire Line
-	10650 2200 10650 3200
-Wire Wire Line
-	10650 2300 10550 2300
-Wire Wire Line
-	10750 3300 10550 3300
-Wire Wire Line
-	10550 2500 10750 2500
-Connection ~ 10650 2300
-$Comp
-L +3.3V #PWR1
+	10550 2600 10750 2600
+Wire Wire Line
+	10750 3400 10550 3400
+Wire Wire Line
+	10650 2700 10550 2700
+Connection ~ 10650 2700
+$Comp
+L +3.3V #PWR024
 U 1 1 53E431FE
-P 10650 2200
-F 0 "#PWR1" H 10650 2160 30  0001 C CNN
-F 1 "+3.3V" H 10650 2310 30  0000 C CNN
-F 2 "~" H 10650 2200 60  0000 C CNN
-F 3 "~" H 10650 2200 60  0000 C CNN
-	1    10650 2200
-	1    0    0    -1
-$EndComp
-Wire Wire Line
-	10750 2200 10750 3300
-$Comp
-L +5V #PWR2
+P 10650 2500
+F 0 "#PWR024" H 10650 2460 30  0001 C CNN
+F 1 "+3.3V" H 10650 2610 30  0000 C CNN
+F 2 "~" H 10650 2500 60  0000 C CNN
+F 3 "~" H 10650 2500 60  0000 C CNN
+	1    10650 2500
+	1    0    0    -1
+$EndComp
+$Comp
+L +5V #PWR025
 U 1 1 53E4332C
-P 10750 2200
-F 0 "#PWR2" H 10750 2290 20  0001 C CNN
-F 1 "+5V" H 10750 2290 30  0000 C CNN
-F 2 "~" H 10750 2200 60  0000 C CNN
-F 3 "~" H 10750 2200 60  0000 C CNN
-	1    10750 2200
-	1    0    0    -1
-$EndComp
-Connection ~ 10750 2500
-Connection ~ 10600 3000
-$Comp
-L GND #PWR13
-U 1 1 53E4357A
-P 10600 3400
-F 0 "#PWR13" H 10600 3400 30  0001 C CNN
-F 1 "GND" H 10600 3330 30  0001 C CNN
-F 2 "~" H 10600 3400 60  0000 C CNN
-F 3 "~" H 10600 3400 60  0000 C CNN
-	1    10600 3400
-	1    0    0    -1
-$EndComp
-NoConn ~ 9400 3400
-NoConn ~ 9400 3500
-NoConn ~ 9400 3600
-NoConn ~ 9400 3700
+P 10750 2550
+F 0 "#PWR025" H 10750 2640 20  0001 C CNN
+F 1 "+5V" H 10750 2640 30  0000 C CNN
+F 2 "~" H 10750 2550 60  0000 C CNN
+F 3 "~" H 10750 2550 60  0000 C CNN
+	1    10750 2550
+	1    0    0    -1
+$EndComp
 NoConn ~ 2050 3800
 NoConn ~ 2050 3900
@@
 	1    0    0    -1
 $EndComp
+Wire Wire Line
+	10750 2550 10750 3400
+Wire Wire Line
+	10650 2500 10650 3500
+Wire Wire Line
+	10650 3500 10550 3500
+Connection ~ 10750 2600
+Wire Wire Line
+	10550 2900 10800 2900
+Wire Wire Line
+	10800 2900 10800 3750
+Wire Wire Line
+	10550 3700 10800 3700
+Connection ~ 10800 3700
+$Comp
+L GND #PWR026
+U 1 1 53E56309
+P 10800 3750
+F 0 "#PWR026" H 10800 3750 30  0001 C CNN
+F 1 "GND" H 10800 3680 30  0001 C CNN
+F 2 "~" H 10800 3750 60  0000 C CNN
+F 3 "~" H 10800 3750 60  0000 C CNN
+	1    10800 3750
+	1    0    0    -1
+$EndComp
+$Comp
+L PAPILIO_WINGS PAP1
+U 1 1 53E3DC81
+P 9950 3100
+F 0 "PAP1" H 9900 3850 60  0000 C CNN
+F 1 "PAPILIO_WINGS" H 9950 3950 60  0000 C CNN
+F 2 "~" H 9600 3950 60  0000 C CNN
+F 3 "~" H 9600 3950 60  0000 C CNN
+	1    9950 3100
+	1    0    0    1
+$EndComp
 $EndSCHEMATC
