File: CODEC Wing/ADC.sch (KiCad schematic (older format))
At the start: 11 parts, among them J2 JACK_ST_2SW_PROPER

Commit message: More stuff
Parts:
- added TP3, TP4: CONN_1, symbol CONN_1
Connections:
- net at ADC1.14 (Vin_R), C13.1, R3.1: now also TP3.1
- net at ADC1.13 (Vin_L), C14.1, R4.1: now also TP4.1
Changed lines of the file:
@@
 Sheet 4 4
 Title "CODEC Wing"
-Date "1 sep 2014"
+Date "2 sep 2014"
 Rev "1.0"
 Comp "Cholula Audio"
@@
 $EndComp
 $Comp
-L +5V #PWR020
+L +5V #PWR21
 U 1 1 5404F3B3
 P 4850 2550
-F 0 "#PWR020" H 4850 2640 20  0001 C CNN
+F 0 "#PWR21" H 4850 2640 20  0001 C CNN
 F 1 "+5V" H 4850 2640 30  0000 C CNN
 F 2 "~" H 4850 2550 60  0000 C CNN
@@
 Connection ~ 4850 3100
 $Comp
-L GND #PWR021
+L GND #PWR23
 U 1 1 5404F3F2
 P 4850 3150
-F 0 "#PWR021" H 4850 3150 30  0001 C CNN
+F 0 "#PWR23" H 4850 3150 30  0001 C CNN
 F 1 "GND" H 4850 3080 30  0001 C CNN
 F 2 "~" H 4850 3150 60  0000 C CNN
@@
 Connection ~ 4050 3500
 $Comp
-L GND #PWR022
+L GND #PWR25
 U 1 1 5404F48A
 P 3750 3550
-F 0 "#PWR022" H 3750 3550 30  0001 C CNN
+F 0 "#PWR25" H 3750 3550 30  0001 C CNN
 F 1 "GND" H 3750 3480 30  0001 C CNN
 F 2 "~" H 3750 3550 60  0000 C CNN
@@
 	8050 2550 8300 2550
 $Comp
-L GND #PWR023
+L GND #PWR22
 U 1 1 5404DA6A
 P 8800 3000
-F 0 "#PWR023" H 8800 3000 30  0001 C CNN
+F 0 "#PWR22" H 8800 3000 30  0001 C CNN
 F 1 "GND" H 8800 2930 30  0001 C CNN
 F 2 "~" H 8800 3000 60  0000 C CNN
@@
 	7600 2850 7650 2850
 Wire Wire Line
-	6700 2950 6700 2550
+	6700 2150 6700 2950
 Wire Wire Line
 	6300 2550 7100 2550
@@
 Connection ~ 6950 3400
 $Comp
-L GND #PWR024
+L GND #PWR24
 U 1 1 5404DD71
 P 6950 3450
-F 0 "#PWR024" H 6950 3450 30  0001 C CNN
+F 0 "#PWR24" H 6950 3450 30  0001 C CNN
 F 1 "GND" H 6950 3380 30  0001 C CNN
 F 2 "~" H 6950 3450 60  0000 C CNN
@@
 $EndComp
 $Comp
-L +3,3V #PWR025
+L +3,3V #PWR20
 U 1 1 5404F26B
 P 4750 2550
-F 0 "#PWR025" H 4750 2510 30  0001 C CNN
+F 0 "#PWR20" H 4750 2510 30  0001 C CNN
 F 1 "+3,3V" H 4750 2660 30  0000 C CNN
 F 2 "~" H 4750 2550 60  0000 C CNN
@@
 	1    0    0    -1
 $EndComp
+$Comp
+L CONN_1 TP4
+U 1 1 5406159D
+P 7100 2300
+F 0 "TP4" H 7180 2300 40  0000 L CNN
+F 1 "CONN_1" H 7100 2355 30  0001 C CNN
+F 2 "" H 7100 2300 60  0000 C CNN
+F 3 "" H 7100 2300 60  0000 C CNN
+	1    7100 2300
+	1    0    0    -1
+$EndComp
+$Comp
+L CONN_1 TP3
+U 1 1 540615AF
+P 7100 2150
+F 0 "TP3" H 7180 2150 40  0000 L CNN
+F 1 "CONN_1" H 7100 2205 30  0001 C CNN
+F 2 "" H 7100 2150 60  0000 C CNN
+F 3 "" H 7100 2150 60  0000 C CNN
+	1    7100 2150
+	1    0    0    -1
+$EndComp
+Wire Wire Line
+	6950 2300 6900 2300
+Wire Wire Line
+	6900 2300 6900 2850
+Connection ~ 6900 2850
+Wire Wire Line
+	6950 2150 6700 2150
+Wire Notes Line
+	6850 2050 6850 2350
+Wire Notes Line
+	6850 2350 7400 2350
+Wire Notes Line
+	7400 2350 7400 2050
+Wire Notes Line
+	7400 2050 6850 2050
 $EndSCHEMATC

Commit message: CODEC Wing
Parts:
- C11, C12: value CP1 -> 1uF
- C13, C14: value C -> 1.5nF
- C15, C16, C17: value CP1 -> 10uF
- R3, R4: value R -> 560R
Changed lines of the file:
@@
 Sheet 4 4
 Title "CODEC Wing"
-Date "2 sep 2014"
+Date "23 sep 2014"
 Rev "1.0"
 Comp "Cholula Audio"
@@
 P 4350 3200
 F 0 "C17" H 4400 3300 50  0000 L CNN
-F 1 "CP1" H 4400 3100 50  0000 L CNN
+F 1 "10uF" H 4400 3100 50  0000 L CNN
 F 2 "~" H 4350 3200 60  0000 C CNN
 F 3 "~" H 4350 3200 60  0000 C CNN
@@
 P 4050 3200
 F 0 "C16" H 4100 3300 50  0000 L CNN
-F 1 "CP1" H 4100 3100 50  0000 L CNN
+F 1 "10uF" H 4100 3100 50  0000 L CNN
 F 2 "~" H 4050 3200 60  0000 C CNN
 F 3 "~" H 4050 3200 60  0000 C CNN
@@
 P 3750 3200
 F 0 "C15" H 3800 3300 50  0000 L CNN
-F 1 "CP1" H 3800 3100 50  0000 L CNN
+F 1 "10uF" H 3800 3100 50  0000 L CNN
 F 2 "~" H 3750 3200 60  0000 C CNN
 F 3 "~" H 3750 3200 60  0000 C CNN
@@
 P 7850 2550
 F 0 "C11" H 7900 2650 50  0000 L CNN
-F 1 "CP1" H 7900 2450 50  0000 L CNN
+F 1 "1uF" H 7900 2450 50  0000 L CNN
 F 2 "~" H 7850 2550 60  0000 C CNN
 F 3 "~" H 7850 2550 60  0000 C CNN
@@
 P 7850 2850
 F 0 "C12" H 7900 2950 50  0000 L CNN
-F 1 "CP1" H 7900 2750 50  0000 L CNN
+F 1 "1uF" H 7900 2750 50  0000 L CNN
 F 2 "~" H 7850 2850 60  0000 C CNN
 F 3 "~" H 7850 2850 60  0000 C CNN
@@
 P 6700 3150
 F 0 "C13" H 6700 3250 40  0000 L CNN
-F 1 "C" H 6706 3065 40  0000 L CNN
+F 1 "1.5nF" H 6706 3065 40  0000 L CNN
 F 2 "~" H 6738 3000 30  0000 C CNN
 F 3 "~" H 6700 3150 60  0000 C CNN
@@
 P 6950 3150
 F 0 "C14" H 6950 3250 40  0000 L CNN
-F 1 "C" H 6956 3065 40  0000 L CNN
+F 1 "1.5nF" H 6956 3065 40  0000 L CNN
 F 2 "~" H 6988 3000 30  0000 C CNN
 F 3 "~" H 6950 3150 60  0000 C CNN
@@
 P 7350 2550
 F 0 "R3" V 7430 2550 40  0000 C CNN
-F 1 "R" V 7357 2551 40  0000 C CNN
+F 1 "560R" V 7357 2551 40  0000 C CNN
 F 2 "~" V 7280 2550 30  0000 C CNN
 F 3 "~" H 7350 2550 30  0000 C CNN
@@
 P 7350 2850
 F 0 "R4" V 7430 2850 40  0000 C CNN
-F 1 "R" V 7357 2851 40  0000 C CNN
+F 1 "560R" V 7357 2851 40  0000 C CNN
 F 2 "~" V 7280 2850 30  0000 C CNN
 F 3 "~" H 7350 2850 30  0000 C CNN
