File: CODEC Wing/CODEC Wing.sch (KiCad schematic (older format))
At the start: 3 parts

Commit message: More stuff
Changed lines of the file:
@@
 Sheet 1 4
 Title "CODEC Wing"
-Date "1 sep 2014"
+Date "2 sep 2014"
 Rev "1.0"
 Comp "Cholula Audio"
@@
 	9700 4550 9700 4500
 $Comp
-L +3.3V #PWR01
+L +3.3V #PWR7
 U 1 1 5404D24E
 P 9700 4500
-F 0 "#PWR01" H 9700 4460 30  0001 C CNN
+F 0 "#PWR7" H 9700 4460 30  0001 C CNN
 F 1 "+3.3V" H 9700 4610 30  0000 C CNN
 F 2 "~" H 9700 4500 60  0000 C CNN
@@
 	9550 4350 9550 4400
 $Comp
-L GND #PWR02
+L GND #PWR6
 U 1 1 5404D291
 P 9550 4400
-F 0 "#PWR02" H 9550 4400 30  0001 C CNN
+F 0 "#PWR6" H 9550 4400 30  0001 C CNN
 F 1 "GND" H 9550 4330 30  0001 C CNN
 F 2 "~" H 9550 4400 60  0000 C CNN
@@
 	9200 3100 9200 3050
 $Comp
-L +5V #PWR03
+L +5V #PWR4
 U 1 1 5404ED22
 P 9200 3050
-F 0 "#PWR03" H 9200 3140 20  0001 C CNN
+F 0 "#PWR4" H 9200 3140 20  0001 C CNN
 F 1 "+5V" H 9200 3140 30  0000 C CNN
 F 2 "~" H 9200 3050 60  0000 C CNN
@@
 	9400 2800 9400 2900
 $Comp
-L GND #PWR04
+L GND #PWR3
 U 1 1 5404ED89
 P 9400 2900
-F 0 "#PWR04" H 9400 2900 30  0001 C CNN
+F 0 "#PWR3" H 9400 2900 30  0001 C CNN
 F 1 "GND" H 9400 2830 30  0001 C CNN
 F 2 "~" H 9400 2900 60  0000 C CNN
@@
 	1600 2950 1600 2900
 $Comp
-L +5V #PWR05
+L +5V #PWR2
 U 1 1 5404E846
 P 1600 2900
-F 0 "#PWR05" H 1600 2990 20  0001 C CNN
+F 0 "#PWR2" H 1600 2990 20  0001 C CNN
 F 1 "+5V" H 1600 2990 30  0000 C CNN
 F 2 "~" H 1600 2900 60  0000 C CNN
@@
 	1500 3250 1500 3300
 $Comp
-L GND #PWR06
+L GND #PWR5
 U 1 1 5404E8DE
 P 1500 3300
-F 0 "#PWR06" H 1500 3300 30  0001 C CNN
+F 0 "#PWR5" H 1500 3300 30  0001 C CNN
 F 1 "GND" H 1500 3230 30  0001 C CNN
 F 2 "~" H 1500 3300 60  0000 C CNN
@@
 $EndSheet
 $Comp
-L +3,3V #PWR07
+L +3,3V #PWR1
 U 1 1 5404F45D
 P 1450 2900
-F 0 "#PWR07" H 1450 2860 30  0001 C CNN
+F 0 "#PWR1" H 1450 2860 30  0001 C CNN
 F 1 "+3,3V" H 1450 3010 30  0000 C CNN
 F 2 "~" H 1450 2900 60  0000 C CNN
@@
 	1    0    0    -1
 $EndComp
-$Comp
-L OSHW #G1
-U 1 1 54050EC4
-P 10550 6300
-F 0 "#G1" H 10550 5820 60  0001 C CNN
-F 1 "OSHW" H 10550 6780 60  0001 C CNN
-F 2 "" H 10550 6300 60  0000 C CNN
-F 3 "" H 10550 6300 60  0000 C CNN
-	1    10550 6300
-	1    0    0    -1
-$EndComp
