File: CODEC Wing/DAC.sch (KiCad schematic (older format))
At the start: 9 parts, among them J1 JACK_ST_2SW_PROPER, U1 TL082

Commit message: More stuff
Parts:
- added TP1, TP2: CONN_1, symbol CONN_1
Connections:
- net at DAC1.7 (Vout_L), R1.1: now also TP1.1
- net at DAC1.8 (Vout_R), R2.1: now also TP2.1
Changed lines of the file:
@@
 Sheet 3 4
 Title "CODEC Wing"
-Date "1 sep 2014"
+Date "2 sep 2014"
 Rev "1.0"
 Comp "Cholula Audio"
@@
 Connection ~ 3450 3450
 $Comp
-L GND #PWR010
+L GND #PWR18
 U 1 1 5404D6C1
 P 3450 3550
-F 0 "#PWR010" H 3450 3550 30  0001 C CNN
+F 0 "#PWR18" H 3450 3550 30  0001 C CNN
 F 1 "GND" H 3450 3480 30  0001 C CNN
 F 2 "~" H 3450 3550 60  0000 C CNN
@@
 	3550 1800 3550 1700
 $Comp
-L +5V #PWR011
+L +5V #PWR10
 U 1 1 5404D6D8
 P 3550 1700
-F 0 "#PWR011" H 3550 1790 20  0001 C CNN
+F 0 "#PWR10" H 3550 1790 20  0001 C CNN
 F 1 "+5V" H 3550 1790 30  0000 C CNN
 F 2 "~" H 3550 1700 60  0000 C CNN
@@
 	3650 3850 3650 3950
 $Comp
-L GND #PWR012
+L GND #PWR19
 U 1 1 5404D712
 P 3650 3950
-F 0 "#PWR012" H 3650 3950 30  0001 C CNN
+F 0 "#PWR19" H 3650 3950 30  0001 C CNN
 F 1 "GND" H 3650 3880 30  0001 C CNN
 F 2 "~" H 3650 3950 60  0000 C CNN
@@
 	2500 2750 2900 2750
 $Comp
-L GND #PWR013
+L GND #PWR14
 U 1 1 5404D75D
 P 2500 2850
-F 0 "#PWR013" H 2500 2850 30  0001 C CNN
+F 0 "#PWR14" H 2500 2850 30  0001 C CNN
 F 1 "GND" H 2500 2780 30  0001 C CNN
 F 2 "~" H 2500 2850 60  0000 C CNN
@@
 Connection ~ 7700 3000
 $Comp
-L GND #PWR014
+L GND #PWR16
 U 1 1 5404D9C3
 P 7700 3300
-F 0 "#PWR014" H 7700 3300 30  0001 C CNN
+F 0 "#PWR16" H 7700 3300 30  0001 C CNN
 F 1 "GND" H 7700 3230 30  0001 C CNN
 F 2 "~" H 7700 3300 60  0000 C CNN
@@
 	4300 1750 4300 1800
 $Comp
-L GND #PWR015
+L GND #PWR11
 U 1 1 5404EEC8
 P 4300 1800
-F 0 "#PWR015" H 4300 1800 30  0001 C CNN
+F 0 "#PWR11" H 4300 1800 30  0001 C CNN
 F 1 "GND" H 4300 1730 30  0001 C CNN
 F 2 "~" H 4300 1800 60  0000 C CNN
@@
 U 1 1 5404EF72
 P 4700 2650
-F 0 "R1" V 4780 2650 40  0000 C CNN
+F 0 "R1" V 4650 2850 40  0000 C CNN
 F 1 "7.15k" V 4707 2651 40  0000 C CNN
 F 2 "~" V 4630 2650 30  0000 C CNN
@@
 $EndComp
 Wire Wire Line
-	4300 2750 4400 2750
-Wire Wire Line
-	4400 2750 4400 2650
+	4400 2750 4300 2750
+Wire Wire Line
+	4400 2500 4400 2750
 Wire Wire Line
 	4400 2650 4450 2650
@@
 	4300 2850 4400 2850
 Wire Wire Line
-	4400 2850 4400 2950
+	4400 2850 4400 3100
 Wire Wire Line
 	4400 2950 4450 2950
@@
 	6750 3200 6750 3250
 $Comp
-L GND #PWR016
+L GND #PWR15
 U 1 1 5404F0BA
 P 6750 3250
-F 0 "#PWR016" H 6750 3250 30  0001 C CNN
+F 0 "#PWR15" H 6750 3250 30  0001 C CNN
 F 1 "GND" H 6750 3180 30  0001 C CNN
 F 2 "~" H 6750 3250 60  0000 C CNN
@@
 	6300 1900 6300 1800
 $Comp
-L +5V #PWR017
+L +5V #PWR12
 U 1 1 5404F103
 P 6300 1800
-F 0 "#PWR017" H 6300 1890 20  0001 C CNN
+F 0 "#PWR12" H 6300 1890 20  0001 C CNN
 F 1 "+5V" H 6300 1890 30  0000 C CNN
 F 2 "~" H 6300 1800 60  0000 C CNN
@@
 	5300 2700 5300 2750
 $Comp
-L GND #PWR018
+L GND #PWR13
 U 1 1 5404F1D1
 P 5300 2750
-F 0 "#PWR018" H 5300 2750 30  0001 C CNN
+F 0 "#PWR13" H 5300 2750 30  0001 C CNN
 F 1 "GND" H 5300 2680 30  0001 C CNN
 F 2 "~" H 5300 2750 60  0000 C CNN
@@
 	5300 3400 5300 3450
 $Comp
-L GND #PWR019
+L GND #PWR17
 U 1 1 5404F26F
 P 5300 3450
-F 0 "#PWR019" H 5300 3450 30  0001 C CNN
+F 0 "#PWR17" H 5300 3450 30  0001 C CNN
 F 1 "GND" H 5300 3380 30  0001 C CNN
 F 2 "~" H 5300 3450 60  0000 C CNN
@@
 	1    0    0    -1
 $EndComp
+$Comp
+L CONN_1 TP2
+U 1 1 54061420
+P 4400 3250
+F 0 "TP2" H 4480 3250 40  0000 L CNN
+F 1 "CONN_1" H 4400 3305 30  0001 C CNN
+F 2 "" H 4400 3250 60  0000 C CNN
+F 3 "" H 4400 3250 60  0000 C CNN
+	1    4400 3250
+	0    1    1    0
+$EndComp
+Connection ~ 4400 2950
+$Comp
+L CONN_1 TP1
+U 1 1 54061472
+P 4600 2500
+F 0 "TP1" H 4680 2500 40  0000 L CNN
+F 1 "CONN_1" H 4600 2555 30  0001 C CNN
+F 2 "" H 4600 2500 60  0000 C CNN
+F 3 "" H 4600 2500 60  0000 C CNN
+	1    4600 2500
+	1    0    0    -1
+$EndComp
+Wire Wire Line
+	4450 2500 4400 2500
+Connection ~ 4400 2650
+Wire Notes Line
+	4300 3050 4500 3050
+Wire Notes Line
+	4500 3050 4500 3500
+Wire Notes Line
+	4500 3500 4300 3500
+Wire Notes Line
+	4300 3500 4300 3050
+Wire Notes Line
+	4350 2450 4350 2550
+Wire Notes Line
+	4350 2550 4850 2550
+Wire Notes Line
+	4850 2550 4850 2450
+Wire Notes Line
+	4850 2450 4350 2450
 $EndSCHEMATC
